File: zudo-pd.kicad_pcb (KiCad board)
At the start: 2 copper layers, 75.7 x 96.9 mm, 70 parts, among them J1 USB-C, J2 2541WR-2X08P, J3 2541WR-2X08P, J4 2541WR-2X08P, J5 2541WR-2X08P, J6 1217754-1, J7 1217754-1, J8 1217754-1, J9 1217754-1, U1 CH224D, U2 LM2596S-ADJ, U3 LM2596S-ADJ, U4 LM2596S-ADJ, U6 L7812CD2T-TR, U7 L7805ABD2T-TR, U8 CJ7912_C94173

Commit message: wip
Parts:
- added TP1: +15V USB-PD, TestPoint:TestPoint_Pad_D1.5mm, F.Cu at (196.5, 44.0)
- added TP2: GND, TestPoint:TestPoint_Pad_D1.5mm, F.Cu at (200.0, 44.0)
- added TP3: +13.5V, TestPoint:TestPoint_Pad_D1.5mm, F.Cu at (204.0, 44.0)
- added TP4: +7.5V, TestPoint:TestPoint_Pad_D1.5mm, F.Cu at (220.0, 88.5)
- added TP5: -13.5V, TestPoint:TestPoint_Pad_D1.5mm, F.Cu at (220.0, 120.5)
- moved LED2 60.4 mm to (164.5, 132.2), turned to 90 degrees
- moved LED3 26.1 mm to (167.0, 132.2), turned to 90 degrees
- moved LED4 16.5 mm to (170.0, 132.5)
- moved J9 10.5 mm to (169.0, 57.9)
- moved J7 5.02 mm to (164.0, 57.9)
- moved J8 4.73 mm to (159.0, 57.9)
- moved D3 1.90 mm to (207.0, 92.8)
- moved C4 1.70 mm to (215.0, 90.5)
Routing:
- net Net-(LED2-A): track 2.30 -> 59.4 mm, vias 0 -> 2
- net Net-(LED3-A): track 2.20 -> 23.9 mm
- net Net-(LED4--): track 2.58 -> 20.8 mm
- net +15V -> +13.5V gen: track 136.3 -> 145.8 mm
- net GND: track 18.7 -> 25.2 mm, vias 46 -> 45
- net /DC-DC Conversion/+7.5V OUT: track 104.6 -> 109.8 mm, vias 2 -> 3
- net /DC-DC Conversion/-13.5V OUT: track 117.6 -> 116.5 mm
- net Net-(D3-K): track 29.2 -> 30.0 mm
Other:
- board text added: "+12V"
- board text added: "+13.5V"
- board text added: "+15V USB-PD"
- board text added: "+5V"
- board text added: "+7.5V"
- board text added: "-13.5V"
- board text added: "GND"

Commit message: wip
Parts:
- LED4: footprint zudo-pd:LED0805-R-RD -> zudo-pd:LED0603-RD
- moved LED4 0.56 mm to (169.5, 132.2)
Connections:
- LED4 pad 1: GND -> Net-(LED4-C)
- LED4 pad 2: Net-(LED4--) -> GND
- R9 pad 2: Net-(LED4--) -> Net-(LED4-C)
Routing:
- net Net-(LED4--): track 20.8 -> 0.00 mm
- net Net-(LED4-C): track 0.00 -> 20.5 mm
- net /DC-DC Conversion/-13.5V OUT: track 116.5 -> 129.4 mm
- net /DC-DC Conversion/+13.5V OUT: track 84.1 -> 93.4 mm
Other:
- board text added: "-12V"

Commit message: kicad file updates
Parts:
- added REF**: MountingHole_3.2mm_M3, MountingHole:MountingHole_3.2mm_M3, F.Cu at (72.5, 3.50)
- added REF**: MountingHole_3.2mm_M3, MountingHole:MountingHole_3.2mm_M3, F.Cu at (12.8, 95.5)
- added REF**: MountingHole_3.2mm_M3, MountingHole:MountingHole_3.2mm_M3, F.Cu at (3.50, 3.50)
- added REF**: MountingHole_3.2mm_M3, MountingHole:MountingHole_3.2mm_M3, F.Cu at (35.5, 20.8)
- added REF**: MountingHole_3.2mm_M3, MountingHole:MountingHole_3.2mm_M3, F.Cu at (72.5, 95.5)
- added REF**: MountingHole_3.2mm_M3, MountingHole:MountingHole_3.2mm_M3, F.Cu at (66.8, 90.0)
- added REF**: MountingHole_3.2mm_M3, MountingHole:MountingHole_3.2mm_M3, F.Cu at (19.8, 68.5)
- moved C3 153.3 mm to (63.5, 12.5)
- moved C5 152.7 mm to (53.5, 14.5)
- moved J1 151.6 mm to (38.7, 5.50)
- moved C24 151.3 mm to (54.1, 75.8)
- moved C1 151.1 mm to (46.8, 12.4)
- moved C10 151.1 mm to (40.5, 62.6)
- moved C14 151.1 mm to (20.9, 59.3)
- moved C15 151.1 mm to (35.7, 87.7)
- moved C16 151.1 mm to (49.1, 82.3)
- moved C17 151.1 mm to (33.4, 42.2)
- moved C18 151.1 mm to (35.9, 76.7)
- moved C19 151.1 mm to (49.2, 86.0)
- moved C2 151.1 mm to (46.2, 14.6)
- moved C20 151.1 mm to (32.0, 59.4)
- moved C21 151.1 mm to (27.1, 35.3)
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Routing:
- net -12V rail: track 11.1 -> 190.0 mm, vias 0 -> 4
- net +12V rail: track 12.2 -> 125.3 mm, vias 0 -> 1
- net CV rail: track 0.00 -> 104.6 mm, vias 0 -> 7
- net +5V rail: track 13.3 -> 114.7 mm
- net GATE rail: track 0.00 -> 91.4 mm
- net Net-(LED2-A): track 59.4 -> 65.1 mm
- net GND: track 25.2 -> 30.5 mm, vias 45 -> 46
- net Net-(D1-K): track 40.5 -> 45.6 mm
- net /DC-DC Conversion/-13.5V OUT: track 129.4 -> 131.8 mm
- net Net-(D3-K): track 30.0 -> 32.3 mm
- net Net-(J1-CC2): track 14.9 -> 16.7 mm
- net Net-(J1-CC1): track 9.86 -> 11.7 mm
- net /DC-DC Conversion/+13.5V OUT: track 93.4 -> 91.7 mm
- net /DC-DC Conversion/+7.5V OUT: track 109.8 -> 111.4 mm, vias 3 -> 2
- net Net-(C16-Pad2): track 17.1 -> 18.7 mm
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Other:
- board size 75.7 x 96.9 mm -> 76 x 99 mm
- board text added: "-12V RED!!"
- board text added: ">"
- board text added: "JLCJLCJLCJLC"
- board text added: "RED!! -12V"
- board text added: "zudo-PD v0.1"
