File: zudo-pd.kicad_pcb (KiCad board)
At the start: 2 copper layers, 76 x 99 mm, 82 parts, among them J1 USB-C, J2 2541WR-2X08P, J3 2541WR-2X08P, J4 2541WR-2X08P, J5 2541WR-2X08P, J6 1217754-1, J7 1217754-1, J8 1217754-1, J9 1217754-1, U1 CH224D, U2 LM2596S-ADJ, U3 LM2596S-ADJ, U4 LM2596S-ADJ, U6 L7812CD2T-TR, U7 L7805ABD2T-TR, U8 CJ7912_C94173

Commit message: update pcb
Connections:
- LED3 pad 1: GND -> GND rail
Routing:
- net GND rail: vias 45 -> 46
- net GND: vias 1 -> 0
