File: usb-pd-input.kicad_sch (KiCad schematic)
At the start: 24 parts, among them J1 USB-C, J2 Pogo pads, J3 Pogo pads (debug), Q1 -30V -4A, U1 STUSB4500QTR

Commit message: fix(usb-pd): restore CCDB topology, DNP external Rd, remove D4, add SMAJ20A (#93)
Rows 1-5 of the locked spec from #90 (issue #93):

- Delete D4 (USBLC6-2SC6, C7519): its 6V zener clamped the 15V VBUS rail
  and its internal flow-through carried the CC lines. CC nets now merge
  straight through: CC1 = J1.A5 + U1.2 + R17.1 + R19.2, CC2 = J1.B5 +
  U1.4 + R18.1 + R20.2 (netlist-verified partition match).
- R17/R18 (external 5.1k Rd): DNP + exclude from BOM + exclude from
  position files. Footprints and value kept for bench-option rework.
- R19/R20 pin 2 rewired from GND to CC1/CC2: they are now the fitted
  0R CC1DB<->CC1 / CC2DB<->CC2 links (CCDB debug topology restored).
- Add D5 = SMAJ20A (LCSC C571370, SMA/DO-214AC): cathode -> VBUS_IN,
  anode -> GND, replacing D4's lost VBUS clamp with a 20V-standoff part.
  Symbol cloned from the SMAJ15A_C571368 pattern (pin 1 = C verified
  against TVS1/TVS3 usage) into symbols/zudo-pd.kicad_sym and embedded
  in the sheet. Existing VBUS_IN global label reused for the cathode.

Verification: kicadxml netlist partition diff vs baseline shows exactly
the intended changes; ERC 0 errors before/after (204 vs 202 warnings,
the +2 being the same 'Unspecified pin' class TVS1/TVS3 already carry).
Note: kicad-cli net-name output for GND/'GND rail' and VBUS_OUT/'+15V
-> +13.5V gen' is nondeterministic run-to-run (pre-existing double-
named nets, confirmed on pristine baseline); membership is stable.

Co-Authored-By: Claude Opus 4.8 (1M context) <noreply@anthropic.com>
Parts:
- removed D4: USBLC6-2SC6, zudo-pd:SOT-23-6_L2.9-W1.6-P0.95-LS2.8-BL, symbol zudo-pd:USBLC6-2SC6_C7519
- added D5: SMAJ20A_C571370, zudo-pd:D-FLAT_L4.3-W2.6-LS5.3-RD, symbol zudo-pd:SMAJ20A_C571370
- R17, R18: now not fitted; now left out of the parts list
Connections:
- net GND: now also D5.2 (A); no longer R19.2, R20.2
- net VBUS_IN: now also D5.1 (C)
- net CC1: now reaches J1.A5 (CC1), R17.1
- net CC1: now also R19.2, U1.2 (CC1)
- net CC2: now reaches J1.B5 (CC2), R18.1
- net CC2: now also R20.2, U1.4 (CC2)
