File: boards/board-a/board-a.kicad_sch (KiCad schematic)
At the start: 28 parts, among them J1 USB-TYPE-C-009, J2 PogoPad_1x4_NVM_I2C, J3 PogoPad_1x8_Debug, J4 B6B-XH-A(LF)(SN), Q1 AO3401A, U1 STUSB4500QTR

Commit message: fix: schgen review fixes — board-a TP footprints, robust errors, geometry verifier
- board_a_spec.py: TP1/TP2/TP6 now use zudo-pd:TestPad_D1.5mm (the committed
  house footprint board B already uses) instead of the undeclared stock
  TestPoint: nickname; adopt board B's shared-constant tuple style
- schgen_core.py: SchgenError instead of bare asserts (works under -O, message
  not traceback), check_coverage collects every violation before failing,
  generate() split into _emit_* stages, UTF-8 + context managers on all file
  I/O, shared load_spec_module() for every CLI
- sexp.py: module docstring, UTF-8 load, drop unused re import, one statement
  per line
- gen_schematic.py / verify_netlist.py: argparse + main() + shared loader
- check_baseline.py: consolidate onto schgen_core.load_spec_module
- new verify_geometry.py: independently re-derives pin endpoints from the
  emitted file and checks labels/no-connects/collisions against the spec;
  wired into run_smoke_test.sh with a negative control
- boards/board-a regenerated (only the three TP footprint properties change;
  board-b regen is byte-identical)

Co-Authored-By: Claude Fable 5 <noreply@anthropic.com>
Parts:
- TP1, TP2, TP6: footprint TestPoint:TestPoint_Pad_D1.5mm -> zudo-pd:TestPad_D1.5mm
Changed lines of the file:
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@@
 			)
 		)
-		(property "Footprint" "TestPoint:TestPoint_Pad_D1.5mm"
+		(property "Footprint" "zudo-pd:TestPad_D1.5mm"
 			(at 355.6 50.8 0)
 			(effects
@@
 			)
 		)
-		(property "Footprint" "TestPoint:TestPoint_Pad_D1.5mm"
+		(property "Footprint" "zudo-pd:TestPad_D1.5mm"
 			(at 355.6 76.2 0)
 			(effects
@@
 			)
 		)
-		(property "Footprint" "TestPoint:TestPoint_Pad_D1.5mm"
+		(property "Footprint" "zudo-pd:TestPad_D1.5mm"
 			(at 355.6 101.6 0)
 			(effects
